Commit message: Update kobuki urdf

File: superh-lab-kobuki-slam/kobuki/kobuki_description/urdf/kobuki_gazebo.urdf.xacro (robot description, xacro)
@@ -1,449 +1,299 @@
 <?xml version="1.0"?>
 <robot name="kobuki_sim" xmlns:xacro="http://ros.org/wiki/xacro">
-  <xacro:macro name="kobuki_sim">
-    <gazebo reference="wheel_left_link">
-      <mu1>1.0</mu1>
-      <mu2>1.0</mu2>
-      <kp>1000000.0</kp>
-      <kd>100.0</kd>
-      <minDepth>0.001</minDepth>
-      <maxVel>1.0</maxVel>
-    </gazebo>
-    <gazebo reference="wheel_right_link">
-      <mu1>1.0</mu1>
-      <mu2>1.0</mu2>
-      <kp>1000000.0</kp>
-      <kd>100.0</kd>
-      <minDepth>0.001</minDepth>
-      <maxVel>1.0</maxVel>
-    </gazebo>
-    <gazebo reference="caster_front_link">
-      <mu1>0.0</mu1>
-      <mu2>0.0</mu2>
-      <kp>1000000.0</kp>
-      <kd>100.0</kd>
-      <minDepth>0.001</minDepth>
-      <maxVel>1.0</maxVel>
-    </gazebo>
-    <gazebo reference="caster_back_link">
-      <mu1>0.0</mu1>
-      <mu2>0.0</mu2>
-      <kp>1000000.0</kp>
-      <kd>100.0</kd>
-      <minDepth>0.001</minDepth>
-      <maxVel>1.0</maxVel>
-    </gazebo>
-    <gazebo reference="base_link">
-      <mu1>0.3</mu1>
-      <mu2>0.3</mu2>
-      <sensor type="contact" name="bumpers">
-        <always_on>1</always_on>
-        <update_rate>50.0</update_rate>
-        <visualize>true</visualize>
-        <contact>
-          <collision>base_footprint_fixed_joint_lump__base_collision</collision>
-        </contact>
-      </sensor>
-    </gazebo>
-    <gazebo reference="cliff_sensor_left_link">
-      <sensor type="ray" name="cliff_sensor_left">
-        <always_on>true</always_on>
-        <update_rate>50</update_rate>
-        <visualize>true</visualize>
-        <ray>
-          <scan>
-            <horizontal>
-              <samples>50</samples>
-              <resolution>1.0</resolution>
-              <min_angle>-0.0436</min_angle>  <!-- -2.5 degree -->
-              <max_angle>0.0436</max_angle> <!-- 2.5 degree -->
-            </horizontal>
-<!--            Can't use vertical rays until this bug is resolved: -->
-<!--            https://bitbucket.org/osrf/gazebo/issue/509/vertical-sensor-doesnt-works -->
-<!--               <vertical> -->
-<!--                 <samples>50</samples> -->
-<!--                 <resolution>1.0</resolution> -->
-<!--                 <min_angle>-0.0436</min_angle>  -2.5 degree -->
-<!--                 <max_angle>0.0436</max_angle> 2.5 degree -->
-<!--               </vertical> -->
-          </scan>
-          <range>
-            <min>0.01</min>
-            <max>0.15</max>
-            <resolution>1.0</resolution>
-          </range>
-        </ray>
-      </sensor>
-    </gazebo>
-    <gazebo reference="cliff_sensor_right_link">
-      <sensor type="ray" name="cliff_sensor_right">
-        <always_on>true</always_on>
-        <update_rate>50</update_rate>
-        <visualize>true</visualize>
-        <ray>
-          <scan>
-            <horizontal>
-              <samples>50</samples>
-              <resolution>1.0</resolution>
-              <min_angle>-0.0436</min_angle>  <!-- -2.5 degree -->
-              <max_angle>0.0436</max_angle> <!-- 2.5 degree -->
-            </horizontal>
-<!--            Can't use vertical rays until this bug is resolved: -->
-<!--            https://bitbucket.org/osrf/gazebo/issue/509/vertical-sensor-doesnt-works -->
-<!--               <vertical> -->
-<!--                 <samples>50</samples> -->
-<!--                 <resolution>1.0</resolution> -->
-<!--                 <min_angle>-0.0436</min_angle>  -2.5 degree -->
-<!--                 <max_angle>0.0436</max_angle> 2.5 degree -->
-<!--               </vertical> -->
-          </scan>
-          <range>
-            <min>0.01</min>
-            <max>0.15</max>
-            <resolution>1.0</resolution>
-          </range>
-        </ray>
-      </sensor>
-    </gazebo>
-    <gazebo reference="cliff_sensor_front_link">
-      <sensor type="ray" name="cliff_sensor_front">
-        <always_on>true</always_on>
-        <update_rate>50</update_rate>
-        <visualize>true</visualize>
-        <ray>
-          <scan>
-            <horizontal>
-              <samples>50</samples>
-              <resolution>1.0</resolution>
-              <min_angle>-0.0436</min_angle>  <!-- -2.5 degree -->
-              <max_angle>0.0436</max_angle> <!-- 2.5 degree -->
-            </horizontal>
-<!--               Can't use vertical rays until this bug is resolved: -->
-<!--            https://bitbucket.org/osrf/gazebo/issue/509/vertical-sensor-doesnt-works -->
-<!--               <vertical> -->
-<!--                 <samples>50</samples> -->
-<!--                 <resolution>1.0</resolution> -->
-<!--                 <min_angle>-0.0436</min_angle>  -2.5 degree -->
-<!--                 <max_angle>0.0436</max_angle> 2.5 degree -->
-<!--               </vertical> -->
-          </scan>
-          <range>
-            <min>0.01</min>
-            <max>0.15</max>
-            <resolution>1.0</resolution>
-          </range>
-        </ray>
-      </sensor>
-    </gazebo>
-    <gazebo reference="gyro_link">
-      <sensor type="imu" name="imu">
-      <always_on>true</always_on>
-      <update_rate>50</update_rate>
-      <visualize>false</visualize>
-      <imu>
-          <noise>
-            <type>gaussian</type>
-            <rate>
-              <mean>0.0</mean>
-              <stddev>${0.0014*0.0014}</stddev> <!-- 0.25 x 0.25 (deg/s) -->
-              <bias_mean>0.0</bias_mean>
-              <bias_stddev>0.0</bias_stddev>
-            </rate>
-            <accel> <!-- not used in the plugin and real robot, hence using tutorial values -->
-              <mean>0.0</mean>
-              <stddev>1.7e-2</stddev>
-              <bias_mean>0.1</bias_mean>
-              <bias_stddev>0.001</bias_stddev>
-            </accel>
-          </noise>
-        </imu>
-      </sensor>
-    </gazebo>
-    <gazebo>
-      <plugin name="kobuki_controller" filename="libgazebo_ros_kobuki.so">
-        <publish_tf>1</publish_tf>
-        <left_wheel_joint_name>wheel_left_joint</left_wheel_joint_name>
-        <right_wheel_joint_name>wheel_right_joint</right_wheel_joint_name>
-        <wheel_separation>.230</wheel_separation>
-        <wheel_diameter>0.070</wheel_diameter>
-        <torque>1.0</torque>
-        <velocity_command_timeout>0.6</velocity_command_timeout>
-        <cliff_sensor_left_name>cliff_sensor_left</cliff_sensor_left_name>
-        <cliff_sensor_center_name>cliff_sensor_front</cliff_sensor_center_name>
-        <cliff_sensor_right_name>cliff_sensor_right</cliff_sensor_right_name>
-        <cliff_detection_threshold>0.04</cliff_detection_threshold>
-        <bumper_name>bumpers</bumper_name>
-        <imu_name>imu</imu_name>
-      </plugin>
-    </gazebo>
-    <!-- Astra 1 -->
-   <gazebo reference="camera1_link">
-    <material>Gazebo/Red</material>
-    <sensor type="depth" name="openni_camera1_camera1">
-      <always_on>1</always_on>
-      <visualize>true</visualize>
-      <camera>
-        <horizontal_fov>1.047</horizontal_fov>
-        <image>
-          <width>640</width>
-          <height>480</height>
-          <format>R8G8B8</format>
-        </image>
-        <depth_camera>
-        </depth_camera>
-        <clip>
-          <near>0.1</near>
-          <far>100</far>
-        </clip>
-      </camera>
-      <plugin name="kinect_controller" filename="libgazebo_ros_openni_kinect.so">
-        <alwaysOn>true</alwaysOn>
-        <updateRate>10.0</updateRate>
-        <cameraName>camera1</cameraName>
-        <frameName>camera_depth_frame</frameName>
-        <imageTopicName>rgb/image_raw</imageTopicName>
-        <depthImageTopicName>depth/image_raw</depthImageTopicName>
-        <pointCloudTopicName>depth/points</pointCloudTopicName>
-        <cameraInfoTopicName>rgb/camera_info</cameraInfoTopicName>
-        <depthImageCameraInfoTopicName>depth/camera_info</depthImageCameraInfoTopicName>
-        <pointCloudCutoff>0.4</pointCloudCutoff>
-        <hackBaseline>0.07</hackBaseline>
-        <distortionK1>0.0</distortionK1>
-        <distortionK2>0.0</distortionK2>
-        <distortionK3>0.0</distortionK3>
-        <distortionT1>0.0</distortionT1>
-        <distortionT2>0.0</distortionT2>
-        <CxPrime>0.0</CxPrime>
-        <Cx>0.0</Cx>
-        <Cy>0.0</Cy>
-        <focalLength>0.0</focalLength>
-      </plugin>
-    </sensor>
-  </gazebo>
-   <!-- Astra 2 -->
-   <gazebo reference="camera2_link">
-    <material>Gazebo/Blue</material>
-    <sensor type="depth" name="openni_camera2_camera2">
-      <always_on>1</always_on>
-      <visualize>true</visualize>
-      <camera>
-        <horizontal_fov>1.047</horizontal_fov>
-        <image>
-          <width>640</width>
-          <height>480</height>
-          <format>R8G8B8</format>
-        </image>
-        <depth_camera>
-        </depth_camera>
-        <clip>
-          <near>0.1</near>
-          <far>100</far>
-        </clip>
-      </camera>
-      <plugin name="kinect_controller" filename="libgazebo_ros_openni_kinect.so">
-        <alwaysOn>true</alwaysOn>
-        <updateRate>10.0</updateRate>
-        <cameraName>camera2</cameraName>
-        <frameName>camera_depth_frame</frameName>
-        <imageTopicName>rgb/image_raw</imageTopicName>
-        <depthImageTopicName>depth/image_raw</depthImageTopicName>
-        <pointCloudTopicName>depth/points</pointCloudTopicName>
-        <cameraInfoTopicName>rgb/camera_info</cameraInfoTopicName>
-        <depthImageCameraInfoTopicName>depth/camera_info</depthImageCameraInfoTopicName>
-        <pointCloudCutoff>0.4</pointCloudCutoff>
-        <hackBaseline>0.07</hackBaseline>
-        <distortionK1>0.0</distortionK1>
-        <distortionK2>0.0</distortionK2>
-        <distortionK3>0.0</distortionK3>
-        <distortionT1>0.0</distortionT1>
-        <distortionT2>0.0</distortionT2>
-        <CxPrime>0.0</CxPrime>
-        <Cx>0.0</Cx>
-        <Cy>0.0</Cy>
-        <focalLength>0.0</focalLength>
-      </plugin>
-    </sensor>
-  </gazebo>
-   <!-- lidar -->
-   <gazebo reference="laser">
-    <material>Gazebo/Black</material>
-    <sensor type="gpu_ray" name="head_rplidar_sensor">
-      <pose>0 0 0 0 0 0</pose>
-      <visualize>false</visualize>
-      <update_rate>40</update_rate>
-      <ray>
-        <scan>
-          <horizontal>
-            <samples>360</samples>
-            <resolution>1</resolution>
-            <min_angle>-3.14159265</min_angle>
-            <max_angle>3.14159265</max_angle>
-          </horizontal>
-        </scan>
-        <range>
-          <min>0.2</min>
-          <max>12.0</max>
-          <resolution>0.01</resolution>
-        </range>
-        <noise>
-          <type>gaussian</type>
-          <mean>0.0</mean>
-          <stddev>0.01</stddev>
-        </noise>
-      </ray>
-      <plugin name="gazebo_ros_head_rplidar_controller" filename="libgazebo_ros_gpu_laser.so">
-        <topicName>scan</topicName>
-        <frameName>laser</frameName>
-      </plugin>
-    </sensor>
-  </gazebo>
-   <!-- range fl -->
-   <!-- <gazebo reference="range_fl">
-    <sensor type="ray" name="range_fl">
-      <pose>0 0 0 0 0 0</pose>
-      <update_rate>5</update_rate>
-      <ray>
-        <scan>
-          <horizontal>
-            <samples>5</samples>
-            <resolution>1.0</resolution>
-            <min_angle>-0.05</min_angle>
-            <max_angle>0.05</max_angle>
-          </horizontal>
-          <vertical>
-            <samples>5</samples>
-            <resolution>1</resolution>
-            <min_angle>-0.05</min_angle>
-            <max_angle>0.05</max_angle>
-          </vertical>
-        </scan>
-        <range>
-          <min>0.01</min>
-          <max>0.9</max>
-          <resolution>0.01</resolution>
-        </range>
-      </ray>
-      <plugin filename="libgazebo_ros_range.so" name="gazebo_ros_range">
-        <gaussianNoise>0.005</gaussianNoise>
-        <alwaysOn>true</alwaysOn>
-        <updateRate>5</updateRate>
-        <topicName>range/fl</topicName>
-        <frameName>range_fl</frameName>
-        <fov>0.1</fov>
-        <radiation>ultrasound</radiation>
-      </plugin>
-    </sensor>
-  </gazebo> -->
-   <!-- range fr -->
-  <!-- <gazebo reference="range_fr">
-    <sensor type="ray" name="range_fr">
-      <pose>0 0 0 0 0 0</pose>
-      <update_rate>5</update_rate>
-      <ray>
-        <scan>
-          <horizontal>
-            <samples>5</samples>
-            <resolution>1.0</resolution>
-            <min_angle>-0.05</min_angle>
-            <max_angle>0.05</max_angle>
-          </horizontal>
-          <vertical>
-            <samples>5</samples>
-            <resolution>1</resolution>
-            <min_angle>-0.05</min_angle>
-            <max_angle>0.05</max_angle>
-          </vertical>
-        </scan>
-        <range>
-          <min>0.01</min>
-          <max>0.9</max>
-          <resolution>0.01</resolution>
-        </range>
-      </ray>
-      <plugin filename="libgazebo_ros_range.so" name="gazebo_ros_range">
-        <gaussianNoise>0.005</gaussianNoise>
-        <alwaysOn>true</alwaysOn>
-        <updateRate>5</updateRate>
-        <topicName>range/fr</topicName>
-        <frameName>range_fr</frameName>
-        <fov>0.1</fov>
-        <radiation>ultrasound</radiation>
-      </plugin>
-    </sensor>
-  </gazebo> -->
-   <!-- range rl -->
-  <!-- <gazebo reference="range_rl">
-    <sensor type="ray" name="range_rl">
-      <pose>0 0 0 0 0 0</pose>
-      <update_rate>5</update_rate>
-      <ray>
-        <scan>
-          <horizontal>
-            <samples>5</samples>
-            <resolution>1.0</resolution>
-            <min_angle>-0.05</min_angle>
-            <max_angle>0.05</max_angle>
-          </horizontal>
-          <vertical>
-            <samples>5</samples>
-            <resolution>1</resolution>
-            <min_angle>-0.05</min_angle>
-            <max_angle>0.05</max_angle>
-          </vertical>
-        </scan>
-        <range>
-          <min>0.01</min>
-          <max>0.9</max>
-          <resolution>0.01</resolution>
-        </range>
-      </ray>
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
Commit message: Update urdf robot

File: superh-lab-kobuki-slam/kobuki/kobuki_description/urdf/kobuki.urdf.xacro (robot description, xacro)
@@ -220,5 +220,5 @@
         <joint name="astra1_joint" type="fixed">
             <axis xyz="0 0 0" />
-            <origin xyz="-0.05 0 0.18" rpy="0 0 0"/>
+            <origin xyz="-0.05 0 0.18" rpy="${pi} ${pi} 0"/>
             <parent link="base_link"/>
             <child link="camera1_link"/>
@@ -232,5 +232,5 @@
             </collision>
             <visual>
-                <origin xyz="-0.01 0 -0.03" rpy="1.5707 0 -1.5707"/>
+                <origin xyz="-0.01 0 -0.03" rpy="1.5707 0 1.5707"/>
                 <geometry>
                     <mesh filename="package://kobuki_description/meshes/astra.stl" scale="0.001 0.001 0.001" />

File: superh-lab-kobuki-slam/kobuki/kobuki_description/urdf/kobuki_gazebo.urdf.xacro (robot description, xacro)
@@ -200,5 +200,5 @@
                     <updateRate>10.0</updateRate>
                     <cameraName>camera1</cameraName>
-                    <frameName>camera_depth_frame</frameName>
+                    <frameName>camera1_depth_frame</frameName>
                     <imageTopicName>rgb/image_raw</imageTopicName>
                     <depthImageTopicName>depth/image_raw</depthImageTopicName>
@@ -243,5 +243,5 @@
                     <updateRate>10.0</updateRate>
                     <cameraName>camera2</cameraName>
-                    <frameName>camera_depth_frame</frameName>
+                    <frameName>camera2_depth_frame</frameName>
                     <imageTopicName>rgb/image_raw</imageTopicName>
                     <depthImageTopicName>depth/image_raw</depthImageTopicName>
@@ -266,7 +266,7 @@
         <gazebo reference="laser">
             <material>Gazebo/Black</material>
-            <sensor type="gpu_ray" name="head_rplidar_sensor">
+            <sensor type="ray" name="head_rplidar_sensor">
                 <pose>0 0 0 0 0 0</pose>
-                <visualize>false</visualize>
+                <visualize>true</visualize>
                 <update_rate>40</update_rate>
                 <ray>
@@ -290,5 +290,5 @@
                     </noise>
                 </ray>
-                <plugin name="gazebo_ros_head_rplidar_controller" filename="libgazebo_ros_gpu_laser.so">
+                <plugin name="gazebo_ros_head_rplidar_controller" filename="libgazebo_ros_laser.so">
                     <topicName>scan</topicName>
                     <frameName>laser</frameName>
